Commit message: modify

File: description/urdf/kait_robot_0.urdf (robot description, URDF)
Before this commit: robot kait_robot, 5 links, 4 joints
Joints:
- joint bno055_1_joint: origin xyz=0.05 -0.2 0.3 rpy=3.1415926 0 -1.57079632679 -> xyz=0.05 -0.2 0.3 rpy=3.1415926 0 0

File: description/urdf/kait_robot_0.urdf.xacro (robot description, xacro)
@@ -56,4 +56,5 @@
 		<child link="imu_link"/>
 		<origin xyz="0.05 -0.2 0.3" rpy="${radians(180)} 0 0"/>
+		<!--origin xyz="0.05 -0.2 0.3" rpy="0 0 0"/-->
 	</joint>
 </robot>
